File: pcb/fork-r0/fork-r0.kicad_pcb (KiCad board)
At the start: 2 copper layers, 96.5 x 55 mm, 108 parts, among them J1 Bus, J2 Prog, J3 SD_Card, J4 Composite, J5 VGA, J9 S-video, U1 ICE40UP5K-SG48ITR50, U10 MIC5504-3.3YM5, U11 THS7314D, U2 74AHC00PW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

Commit message: Creating forks
Parts:
- removed LOGO1: X16 logo, vera-module:x16plogo
Other:
- board text added: "jlcjlcjlcjlc"
