File: pcb/fork-r1/fork-r1.kicad_sch (KiCad schematic)
At the start: 80 parts, among them J1 Bus, J2 Prog, J4 Micro_SD_Card_Det1, J5 VGA, U1 ICE40UP5K-SG48ITR50, U10 MIC5504-3.3YM5, U2 74AHC00PW, U3 SN74CBTD3861PWR, U4 74CBTLV3126PW,118, U5 74LVC4245APW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

Commit message: Adding component IDs
Parts:
- C1, C10, C16, C17, C18, C19, C27, C3, C35, C4, C5, C6, C9: LCSC Part # (none) -> C14663
- C11, C12, C2, C22, C37, C7, C8: LCSC Part # (none) -> C19666
- C23, C24, C25, C26: LCSC Part # (none) -> C15850
- L1: LCSC Part # (none) -> C92959
- R1, R2, R3: LCSC Part # (none) -> C25804
- R14, R16, R19, R20, R4, R5, R6, R7, R8, R9: LCSC Part # (none) -> C25819
- R17, R18: LCSC Part # (none) -> C22936
- R21, R31, R39: LCSC Part # (none) -> C17746
- R24, R33, R40: LCSC Part # (none) -> C22762
- R25, R35, R41: LCSC Part # (none) -> C22901
- R27, R38, R42: LCSC Part # (none) -> C137712
- R34, R37: LCSC Part # (none) -> C23253
- U10: LCSC Part # (none) -> C41348078
- U2: LCSC Part # (none) -> C8143
- U5: LCSC Part # (none) -> C354456
- U7: LCSC Part # (none) -> C2456211

Commit message: Improving R1
Parts:
- H1, H2, H3, H4: footprint MountingHole:MountingHole_3.2mm_M3 -> MountingHole:MountingHole_3.2mm_M3_Pad_Via
Changed lines of the file:
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@@
 			)
 		)
-		(property "Footprint" "MountingHole:MountingHole_3.2mm_M3"
+		(property "Footprint" "MountingHole:MountingHole_3.2mm_M3_Pad_Via"
 			(at 88.9 262.89 0)
 			(hide yes)
@@
 			)
 		)
-		(property "Footprint" "MountingHole:MountingHole_3.2mm_M3"
+		(property "Footprint" "MountingHole:MountingHole_3.2mm_M3_Pad_Via"
 			(at 88.9 267.97 0)
 			(hide yes)
@@
 			)
 		)
-		(property "Footprint" "MountingHole:MountingHole_3.2mm_M3"
+		(property "Footprint" "MountingHole:MountingHole_3.2mm_M3_Pad_Via"
 			(at 88.9 273.05 0)
 			(hide yes)
@@
 			)
 		)
-		(property "Footprint" "MountingHole:MountingHole_3.2mm_M3"
+		(property "Footprint" "MountingHole:MountingHole_3.2mm_M3_Pad_Via"
 			(at 88.9 278.13 0)
 			(hide yes)
