File: toolchain/programmer/pcb/vera-programmer.kicad_sch (KiCad schematic)
At the start: 8 parts, among them J1 Conn_02x05_Odd_Even, SW1 SW_Push, U1 Pico

Commit message: Fixing programmer board and updating licensing
Parts:
- removed J1: Conn_02x05_Odd_Even, Connector_IDC:IDC-Header_2x05_P2.54mm_Vertical, symbol Connector_Generic:Conn_02x05_Odd_Even
- removed U1: Pico, MCU_RaspberryPi_and_Boards:RPi_Pico_SMD_TH, symbol MCU_RaspberryPi_and_Boards:Pico
- added A1: RaspberryPi_Pico, Module:RaspberryPi_Pico_Common_Unspecified, symbol MCU_Module:RaspberryPi_Pico
- added D2: READ, LED_THT:LED_D5.0mm, symbol Device:LED
- added D3: WRITE, LED_THT:LED_D5.0mm, symbol Device:LED
- added J1: Prog, Connector_PinHeader_2.54mm:PinHeader_1x08_P2.54mm_Vertical, symbol Connector_Generic:Conn_01x08
- added R2, R3: 560, Resistor_THT:R_Axial_DIN0207_L6.3mm_D2.5mm_P7.62mm_Horizontal, symbol Device:R
- H1, H2, H3, H4: footprint MountingHole:MountingHole_3.2mm_M3_DIN965 -> MountingHole:MountingHole_3.2mm_M3; now in the parts list
- R1: value 10k -> 10K; LCSC (none) -> C17414; LCSC Part # (none) -> C17414
- SW1: value SW_Push -> RESET
Connections:
- net +3V3: now also A1.36 (3V3)
- net +5V: now also A1.39 (VSYS), A1.40 (VBUS), J1.1 (Pin_1)
- net FPGA_CDONE: now also A1.19 (GPIO14), J1.2 (Pin_2)
- net FPGA_CRESET_B: now also A1.20 (GPIO15), J1.3 (Pin_3)
- net GND: now also A1.13 (GND), A1.18 (GND), A1.23 (GND), A1.28 (GND), A1.3 (GND), A1.33 (AGND), A1.38 (GND), A1.8 (GND), J1.8 (Pin_8), R2.2, R3.2
- net RUN: now also A1.30 (RUN)
- net SPI_MISO: now also A1.21 (GPIO16), J1.4 (Pin_4)
- net SPI_MOSI: now also A1.25 (GPIO19), J1.5 (Pin_5)
- net SPI_SCK: now also A1.24 (GPIO18), J1.6 (Pin_6)
- net SPI_SSEL_N: now also A1.22 (GPIO17), J1.7 (Pin_7)
- new net: D3.1 (K), R3.1
- new net: D2.1 (K), R2.1
- new net GPIO26_3v3: A1.31 (GPIO26_ADC0), D2.2 (A)
- new net GPIO27_3v3: A1.32 (GPIO27_ADC1), D3.2 (A)
- no-connect marks 25 -> 20

Commit message: Expanding massively
Parts:
- removed A1: RaspberryPi_Pico, Module:RaspberryPi_Pico_Common_Unspecified, symbol MCU_Module:RaspberryPi_Pico
- added A2: RaspberryPi_Pico, Module:RaspberryPi_Pico_Common_Unspecified, symbol MCU_Module:RaspberryPi_Pico
Connections:
- net +3V3: now also A2.36 (3V3)
- net +5V: now also A2.40 (VBUS)
- net FPGA_CDONE: now also A2.19 (GPIO14)
- net FPGA_CRESET_B: now also A2.20 (GPIO15)
- net GND: now also A2.13 (GND), A2.18 (GND), A2.23 (GND), A2.28 (GND), A2.3 (GND), A2.33 (AGND), A2.38 (GND), A2.8 (GND)
- net GPIO26_3v3: now also A2.31 (GPIO26_ADC0)
- net GPIO27_3v3: now also A2.32 (GPIO27_ADC1)
- net RUN: now also A2.30 (RUN)
- net SPI_MISO: now also A2.21 (GPIO16)
- net SPI_MOSI: now also A2.25 (GPIO19)
- net SPI_SCK: now also A2.24 (GPIO18)
- net SPI_SSEL_N: now also A2.22 (GPIO17)
- no-connect marks 20 -> 22
Changed lines of the file:
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@@
+	)
+	(no_connect
+		(at 54.61 27.94)
 	)
 	(no_connect
@@
 	(no_connect
 		(at 36.83 73.66)
+	)
+	(no_connect
+		(at 97.79 -90.17)
 	)
 	(no_connect
@@
 	)
 	(symbol
+		(lib_id "MCU_Module:RaspberryPi_Pico")
+		(at 59.69 66.04 0)
+		(unit 1)
+		(body_style 1)
+		(exclude_from_sim no)
+		(in_bom yes)
+		(on_board yes)
+		(in_pos_files yes)
+		(dnp no)
+		(fields_autoplaced yes)
+		(property "Reference" "A2"
+			(at 61.8333 100.33 0)
+			(show_name no)
+			(do_not_autoplace no)
+			(effects
+				(font
+					(size 1.27 1.27)
+				)
+				(justify left)
+			)
+		)
+		(property "Value" "RaspberryPi_Pico"
+			(at 61.8333 102.87 0)
+			(show_name no)
+			(do_not_autoplace no)
+			(effects
+				(font
+					(size 1.27 1.27)
+				)
+				(justify left)
+			)
+		)
+		(property "Footprint" "Module:RaspberryPi_Pico_Common_Unspecified"
+			(at 59.69 113.03 0)
+			(hide yes)
+			(show_name no)
+			(do_not_autoplace no)
+			(effects
+				(font
+					(size 1.27 1.27)
+				)
+			)
+		)
+		(property "Datasheet" "https://datasheets.raspberrypi.com/pico/pico-datasheet.pdf"
+			(at 59.69 115.57 0)
+			(hide yes)
+			(show_name no)
+			(do_not_autoplace no)
+			(effects
+				(font
+					(size 1.27 1.27)
+				)
+			)
+		)
+		(property "Description" "Versatile and inexpensive microcontroller module powered by RP2040 dual-core Arm Cortex-M0+ processor up to 133 MHz, 264kB SRAM, 2MB QSPI flash; also supports Raspberry Pi Pico 2"
+			(at 59.69 118.11 0)
+			(hide yes)
+			(show_name no)
+			(do_not_autoplace no)
+			(effects
+				(font
+					(size 1.27 1.27)
+				)
+			)
+		)
+		(pin "21"
+		)
+		(pin "19"
+		)
+		(pin "24"
+		)
+		(pin "6"
+		)
+		(pin "13"
+		)
+		(pin "1"
+		)
+		(pin "11"
+		)
+		(pin "16"
+		)
+		(pin "31"
+		)
+		(pin "33"
+		)
+		(pin "2"
+		)
+		(pin "5"
+		)
+		(pin "3"
+		)
+		(pin "8"
+		)
+		(pin "10"
+		)
+		(pin "12"
+		)
+		(pin "9"
+		)
+		(pin "4"
+		)
+		(pin "7"
+		)
+		(pin "15"
+		)
+		(pin "17"
+		)
+		(pin "18"
+		)
+		(pin "14"
+		)
+		(pin "20"
+		)
+		(pin "22"
+		)
+		(pin "23"
+		)
+		(pin "26"
+		)
+		(pin "27"
+		)
+		(pin "28"
+		)
+		(pin "29"
+		)
+		(pin "25"
+		)
+		(pin "30"
+		)
+		(pin "32"
+		)
+		(pin "37"
+		)
+		(pin "36"
+		)
+		(pin "40"
+		)
+		(pin "34"
+		)
+		(pin "38"
+		)
+		(pin "35"
+		)
+		(pin "39"
+		)
+		(instances
+			(project "vera-programmer"
+				(path "/f0d61a45-9def-4bf6-bbc4-c71bae198399"
+					(reference "A2")
+					(unit 1)
+				)
+			)
+		)
+	)
+	(symbol
 		(lib_id "Mechanical:MountingHole")
 		(at 21.59 182.88 0)
@@
 	)
 	(symbol
-		(lib_id "power:+5V")
-		(at 54.61 27.94 0)
-		(unit 1)
-		(body_style 1)
-		(exclude_from_sim no)
-		(in_bom yes)
-		(on_board yes)
-		(in_pos_files yes)
-		(dnp no)
-		(fields_autoplaced yes)
-		(property "Reference" "#PWR01"
-			(at 54.61 31.75 0)
-			(hide yes)
-			(show_name no)
-			(do_not_autoplace no)
-			(effects
-				(font
-					(size 1.27 1.27)
-				)
-			)
-		)
-		(property "Value" "+5V"
-			(at 54.61 22.86 0)
-			(show_name no)
-			(do_not_autoplace no)
-			(effects
-				(font
-					(size 1.27 1.27)
-				)
-			)
-		)
-		(property "Footprint" ""
-			(at 54.61 27.94 0)
-			(hide yes)
-			(show_name no)
-			(do_not_autoplace no)
-			(effects
-				(font
-					(size 1.27 1.27)
-				)
-			)
-		)
-		(property "Datasheet" ""
-			(at 54.61 27.94 0)
-			(hide yes)
-			(show_name no)
-			(do_not_autoplace no)
-			(effects
-				(font
-					(size 1.27 1.27)
-				)
-			)
-		)
-		(property "Description" "Power symbol creates a global label with name \"+5V\""
-			(at 54.61 27.94 0)
-			(hide yes)
-			(show_name no)
-			(do_not_autoplace no)
-			(effects
-				(font
-					(size 1.27 1.27)
-				)
-			)
-		)
-		(pin "1"
-		)
-		(instances
-			(project "vera-programmer"
-				(path "/f0d61a45-9def-4bf6-bbc4-c71bae198399"
-					(reference "#PWR01")
-					(unit 1)
-				)
-			)
-		)
-	)
-	(symbol
 		(lib_id "power:GND")
 		(at 132.08 72.39 0)
@@
 					(unit 1)
 				)
-			)
-		)
-	)
-	(symbol
-		(lib_id "MCU_Module:RaspberryPi_Pico")
-		(at 59.69 66.04 0)
-		(unit 1)
-		(body_style 1)
-		(exclude_from_sim no)
-		(in_bom yes)
-		(on_board yes)
-		(in_pos_files yes)
-		(dnp no)
-		(fields_autoplaced yes)
-		(property "Reference" "A1"
-			(at 61.8333 100.33 0)
-			(show_name no)
-			(do_not_autoplace no)
-			(effects
-				(font
-					(size 1.27 1.27)
-				)
-				(justify left)
-			)
-		)
-		(property "Value" "RaspberryPi_Pico"
-			(at 61.8333 102.87 0)
-			(show_name no)
-			(do_not_autoplace no)
-			(effects
-				(font
-					(size 1.27 1.27)
-				)
-				(justify left)
-			)
-		)
-		(property "Footprint" "Module:RaspberryPi_Pico_Common_Unspecified"
-			(at 59.69 113.03 0)
-			(hide yes)
-			(show_name no)
-			(do_not_autoplace no)
-			(effects
-				(font
-					(size 1.27 1.27)
-				)
-			)
-		)
-		(property "Datasheet" "https://datasheets.raspberrypi.com/pico/pico-datasheet.pdf"
-			(at 59.69 115.57 0)
-			(hide yes)
-			(show_name no)
-			(do_not_autoplace no)
-			(effects
-				(font
-					(size 1.27 1.27)
-				)
-			)
-		)
-		(property "Description" "Versatile and inexpensive microcontroller module powered by RP2040 dual-core Arm Cortex-M0+ processor up to 133 MHz, 264kB SRAM, 2MB QSPI flash; also supports Raspberry Pi Pico 2"
-			(at 59.69 118.11 0)
-			(hide yes)
-			(show_name no)
-			(do_not_autoplace no)
-			(effects
-				(font
-					(size 1.27 1.27)
-				)
-			)
-		)
-		(pin "14"
-		)
-		(pin "21"
-		)
-		(pin "18"
-		)
-		(pin "13"
-		)
-		(pin "17"
-		)
-		(pin "15"
-		)
-		(pin "20"
-		)
-		(pin "12"
-		)
-		(pin "25"
-		)
-		(pin "28"
-		)
-		(pin "16"
-		)
-		(pin "24"
-		)
-		(pin "33"
-		)
-		(pin "35"
-		)
-		(pin "38"
-		)
-		(pin "31"
-		)
-		(pin "19"
-		)
-		(pin "26"
-		)
-		(pin "32"
-		)
-		(pin "34"
-		)
-		(pin "22"
-		)
-		(pin "27"
-		)
-		(pin "29"
-		)
-		(pin "23"
-		)
-		(pin "30"
-		)
-		(pin "37"
-		)
-		(pin "39"
-		)
-		(pin "36"
-		)
-		(pin "40"
-		)
-		(pin "6"
-		)
-		(pin "10"
-		)
-		(pin "1"
-		)
-		(pin "8"
-		)
-		(pin "11"
-		)
-		(pin "3"
-		)
-		(pin "7"
-		)
-		(pin "2"
-		)
-		(pin "9"
-		)
-		(pin "4"
-		)
-		(pin "5"
-		)
-		(instances
-			(project "vera-programmer"
-				(path "/f0d61a45-9def-4bf6-bbc4-c71bae198399"
-					(reference "A1")
-					(unit 1)
-				)
